File: work/kicad/demo_p01/demo_p01.kicad_sch (KiCad schematic)
At the start: 14 parts, among them P1 LSI, Q1 3906, U1 JMP

Commit message: Arduino Study at 2022-08-26-[17:28]
Parts:
- removed 0.1uF1: 0.1 uF, symbol 1_KJC_LED_Library:myJac
- removed C1: myJac, symbol 1_KJC_LED_Library:myJac
- removed P1: LSI, symbol Connector:Conn_WallPlug
- removed Q1: 3906, symbol 1_KJC_LED_Library:myJac
- removed R10, R6, R7, R8, R9: 10K, symbol Device:R
- removed S1: A1, symbol Switch:SW_Push
- removed S2: A2, symbol Switch:SW_Push
- removed S3: A3, symbol Switch:SW_Push
- removed S4: RESET, symbol Switch:SW_Push
- removed U1: JMP, symbol 1_KJC_LED_Library:myJMP
- added A?: Arduino_UNO_R3, Module:Arduino_UNO_R3, symbol MCU_Module:Arduino_UNO_R3
- added DS?: WC1602A, Display:WC1602A, symbol Display_Character:WC1602A
